File: CAN_IMU/CAN_IMU.kicad_pcb (KiCad board)
At the start: 2 copper layers, 30 x 65 mm, 45 parts, among them J1 xt30, J2 amazon bno055, J3 bno055 ssci, J4 bno055 ssci, J5 GH2, J6 stlink, U1 TES1-2411, U2 TCAN332G, U3 NJM12888F33, U4 STM32F042K6Tx

Commit message: 一応完成
Parts:
- removed JP2: jump, Jumper:SolderJumper-2_P1.3mm_Open_RoundedPad1.0x1.5mm
- removed REF** (x4): MountingHole_3.2mm_M3, MountingHole:MountingHole_3.2mm_M3
- added C16: 4.7u, Capacitor_SMD:C_0603_1608Metric_Pad1.05x0.95mm_HandSolder, F.Cu at (222.1, 134.0)
- C10: value 4.7u -> 0.1u
- C11, C9: value 0.1u -> 4.7u
- C14: value 0.47u -> 0.1u
- C15: value 4.7u -> 0.47u
- C2: value 1u -> 10u
- C4: value 0.1u -> 1u
- C5: value 5-10u -> 0.1u
- C6: value 0.01u -> 5-10u
- C7: value 1u -> 0.01u
- C8: value 4.7u -> 1u
- moved C5 70.2 mm to (211.0, 134.0), turned to 90 degrees
- moved JP1 66.8 mm to (205.0, 145.2)
- moved D5 62.7 mm to (213.9, 137.5)
- moved R3 60.0 mm to (206.4, 138.2), turned to 180 degrees
- moved R8 57.9 mm to (222.1, 135.5)
- moved R7 57.5 mm to (222.1, 132.5), turned to 180 degrees
- moved R5 57.5 mm to (218.1, 137.5), turned to 180 degrees
- moved C9 56.3 mm to (205.1, 132.0), turned to 180 degrees
- moved D1 56.0 mm to (202.1, 135.2)
- moved C4 55.3 mm to (207.0, 109.5), turned to 90 degrees
- moved R4 54.7 mm to (206.4, 140.8), turned to 180 degrees
- moved R1 54.6 mm to (206.4, 135.2), turned to 180 degrees
- moved R2 49.7 mm to (206.4, 136.8), turned to 180 degrees
- moved D3 48.8 mm to (202.1, 138.2)
- moved C7 47.9 mm to (207.6, 117.5), turned to 180 degrees
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Connections:
- C1 pad 1: +24V -> +5V
- C1 pad 2: GNDPWR -> GND
- C13 pad 1: +5V -> +3V3
- C14 pad 1: +3V3 -> +5V
- C15 pad 1: Net-(C15-Pad1) -> +3V3
- C3 pad 1: +5V -> +24V
- C3 pad 2: GND -> GNDPWR
- C4 pad 1: +3V3 -> +5V
- J1 pad 1: +24V -> GNDPWR
- J1 pad 2: GNDPWR -> +24V
- J3 pad 2: Net-(J3-Pad2) -> (no net)
- JP1 pad 1: +3V3 -> +5V
- JP1 pad 2: Net-(J3-Pad2) -> Net-(J3-Pad6)
- R7 pad 2: Net-(C15-Pad1) -> Net-(C16-Pad1)
- R8 pad 1: Net-(C15-Pad1) -> Net-(C16-Pad1)
- U4 pad 12: (no net) -> /LED_B
- U4 pad 13: (no net) -> /LED_G
- U4 pad 14: (no net) -> /LED_R
- U4 pad 6: /LED_R -> (no net)
- U4 pad 7: /LED_G -> (no net)
- U4 pad 8: /LED_B -> (no net)
Routing:
- net +3V3: track 0.00 -> 89.5 mm, vias 0 -> 9
- net +5V: track 0.00 -> 87.9 mm, vias 0 -> 6
- net GND: track 0.00 -> 74.5 mm, vias 0 -> 63
- net GNDPWR: track 0.00 -> 27.5 mm
- net SDA: track 0.00 -> 27.5 mm, vias 0 -> 2
- net SCL: track 0.00 -> 26.0 mm, vias 0 -> 2
- net +24V: track 0.00 -> 20.5 mm
- net /LED_B: track 0.00 -> 18.8 mm, vias 0 -> 2
- net /LED_G: track 0.00 -> 16.1 mm, vias 0 -> 2
- net SWCLK: track 0.00 -> 15.1 mm, vias 0 -> 1
- net RESET: track 0.00 -> 14.9 mm, vias 0 -> 3
- net /LED_R: track 0.00 -> 13.7 mm, vias 0 -> 2
- net CAN_RX: track 0.00 -> 12.5 mm, vias 0 -> 2
- net SWDIO: track 0.00 -> 12.0 mm, vias 0 -> 1
- net CAN_H: track 0.00 -> 8.95 mm
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- added copper zone on B.Cu, net +3V3
- added copper zone on F.Cu, net +3V3
- added copper zone on B.Cu, net +5V
- added copper zone on F.Cu, net +5V
- added copper zone on B.Cu, net GND
- added copper zone on F.Cu, net GND
Other:
- outline, holes or cut-outs redrawn
- board text added: "3.3V on"
- board text added: "3V3 SWCLK GND SWDIO RESET XXX"
- board text added: "5V"
- board text added: "GND"
- board text added: "R G B"
- board text added: "SCL"
- board text added: "SDA"
- board text added: "termination resistor"
